File: bldc_driver.sch (EAGLE design)
At the start: 42 parts, among them Q1 MOSFET-N, Q2 MOSFET-N, Q3 MOSFET-N, Q4 MOSFET-N, Q5 MOSFET-N, Q6 MOSFET-N, X1 LOGIC, X3 MICROMATCH-10

Commit message: Changed hall sensor connections to proper order
Connections:
- net H1: now also MOTOR.10; no longer MOTOR.9
- net H2: now also MOTOR.9; no longer MOTOR.8
- net H3: now also MOTOR.8; no longer MOTOR.10
Changed lines of the file:
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@@
 <net name="H2" class="0">
+<segment>
+<pinref part="DRV" gate="G$1" pin="H2"/>
+<wire x1="17.78" y1="50.8" x2="7.62" y2="50.8" width="0.1524" layer="91"/>
+<label x="7.62" y="50.8" size="1.778" layer="95"/>
+</segment>
+<segment>
+<pinref part="MOTOR" gate="A" pin="9"/>
+<wire x1="208.28" y1="43.18" x2="200.66" y2="43.18" width="0.1524" layer="91"/>
+<label x="200.66" y="43.18" size="1.778" layer="95"/>
+</segment>
+</net>
+<net name="H1" class="0">
+<segment>
+<pinref part="DRV" gate="G$1" pin="H1"/>
+<wire x1="17.78" y1="53.34" x2="7.62" y2="53.34" width="0.1524" layer="91"/>
+<label x="7.62" y="53.34" size="1.778" layer="95"/>
+</segment>
+<segment>
+<pinref part="MOTOR" gate="A" pin="10"/>
+<wire x1="208.28" y1="40.64" x2="200.66" y2="40.64" width="0.1524" layer="91"/>
+<label x="200.66" y="40.64" size="1.778" layer="95"/>
+</segment>
+</net>
+<net name="H3" class="0">
+<segment>
+<pinref part="DRV" gate="G$1" pin="H3"/>
+<wire x1="17.78" y1="48.26" x2="7.62" y2="48.26" width="0.1524" layer="91"/>
+<label x="7.62" y="48.26" size="1.778" layer="95"/>
+</segment>
 <segment>
 <pinref part="MOTOR" gate="A" pin="8"/>
@@
 <label x="200.66" y="45.72" size="1.778" layer="95"/>
 </segment>
-<segment>
-<pinref part="DRV" gate="G$1" pin="H2"/>
-<wire x1="17.78" y1="50.8" x2="7.62" y2="50.8" width="0.1524" layer="91"/>
-<label x="7.62" y="50.8" size="1.778" layer="95"/>
-</segment>
 </net>
-<net name="H1" class="0">
-<segment>
-<pinref part="MOTOR" gate="A" pin="9"/>
-<wire x1="208.28" y1="43.18" x2="200.66" y2="43.18" width="0.1524" layer="91"/>
-<label x="200.66" y="43.18" size="1.778" layer="95"/>
-</segment>
-<segment>
-<pinref part="DRV" gate="G$1" pin="H1"/>
-<wire x1="17.78" y1="53.34" x2="7.62" y2="53.34" width="0.1524" layer="91"/>
-<label x="7.62" y="53.34" size="1.778" layer="95"/>
-</segment>
-</net>
-<net name="H3" class="0">
-<segment>
-<pinref part="MOTOR" gate="A" pin="10"/>
-<wire x1="208.28" y1="40.64" x2="200.66" y2="40.64" width="0.1524" layer="91"/>
-<label x="200.66" y="40.64" size="1.778" layer="95"/>
-</segment>
-<segment>
-<pinref part="DRV" gate="G$1" pin="H3"/>
-<wire x1="17.78" y1="48.26" x2="7.62" y2="48.26" width="0.1524" layer="91"/>
-<label x="7.62" y="48.26" size="1.778" layer="95"/>
-</segment>
-</net>
